File: version 1 - QMK Proton C/matrix.sch (KiCad schematic (older format))
At the start: 196 parts

Commit message: footprint assignments
Proton C didn't have a footprint available, will need to create a footprint with pin array
Parts:
- D1, D10, D11, D12, D13, D14, D15, D16, D17, D18, D19, D2, D20, D21, D22, D23, D24, D25, D26, D27, D28, D29, D3, D30, D31, D32, D33, D34, D35, D36, D37, D38, D39, D4, D40, D41, D42, D43, D44, D45, D46, D47, D48, D49, D5, D50, D51, D52, D53, D54, D55, D56, D57, D58, D59, D6, D60, D61, D62, D63, D64, D65, D66, D67, D68, D69, D7, D70, D71, D72, D73, D74, D75, D76, D77, D78, D79, D8, D80, D81, D82, D83, D84, D85, D86, D87, D88, D89, D9, D90, D91, D92, D93, D94, D95, D96, D97, D98: footprint (none) -> Diode_SMD:D_SOD-123
- MX1, MX10, MX11, MX12, MX13, MX15, MX16, MX17, MX18, MX19, MX2, MX20, MX21, MX22, MX23, MX24, MX25, MX26, MX27, MX28, MX29, MX3, MX30, MX31, MX33, MX34, MX35, MX36, MX38, MX39, MX4, MX40, MX41, MX42, MX43, MX44, MX45, MX46, MX47, MX48, MX49, MX5, MX51, MX52, MX53, MX54, MX56, MX57, MX58, MX59, MX6, MX60, MX61, MX62, MX63, MX64, MX65, MX66, MX68, MX69, MX7, MX70, MX71, MX73, MX74, MX75, MX76, MX77, MX78, MX79, MX8, MX80, MX81, MX82, MX84, MX85, MX86, MX87, MX9, MX95, MX96, MX97, MX98: footprint (none) -> MX_Alps_Hybrid:MX-1U-NoLED
- MX14, MX37, MX50, MX83: footprint (none) -> MX_Alps_Hybrid:MX-1.5U-NoLED
- MX32, MX88: footprint (none) -> MX_Alps_Hybrid:MX-2U-NoLED
- MX55: footprint (none) -> MX_Alps_Hybrid:MX-1.75U-NoLED
- MX67, MX72: footprint (none) -> MX_Alps_Hybrid:MX-2.25U-NoLED
- MX89, MX90, MX91, MX93, MX94: footprint (none) -> MX_Alps_Hybrid:MX-1.25U-NoLED
- MX92: footprint (none) -> MX_Alps_Hybrid:MX-6.25U-NoLED
