File: version 2 - STM32F303VC no RGB/matrix.sch (KiCad schematic (older format))
At the start: 196 parts

Commit message: switch and diode layout done
Parts:
- MX98: footprint MX_Alps_Hybrid:MX-1U-NoLED -> MX_Alps_Hybrid:MX-2U-NoLED
Changed lines of the file:
@@
 F 0 "MX98" H 8733 5273 60  0000 C CNN
 F 1 "NUM0" H 8733 5199 20  0000 C CNN
-F 2 "MX_Alps_Hybrid:MX-1U-NoLED" H 8075 5025 60  0001 C CNN
+F 2 "MX_Alps_Hybrid:MX-2U-NoLED" H 8075 5025 60  0001 C CNN
 F 3 "" H 8075 5025 60  0001 C CNN
 	1    8700 5050
