File: version 2 - STM32F303VC no RGB/_autosave-GCS98v2.kicad_pcb (KiCad board)
At the start: 2 copper layers, 201 parts, among them SW1 SW_Push, SW2 SW_Push_SPDT, U1 STM32F303CCTx

Commit message: project corrupted
system event viewer: "The description for Event ID 1 from source NVIDIA OpenGL Driver cannot be found. Either the component that raises this event is not installed on your local computer or the installation is corrupted. You can install or repair the component on the local computer."

rolling back to previous commit after submitting this one
Routing:
- net col05: track 109.7 -> 125.1 mm
- net col04: track 90.6 -> 91.8 mm
Other:
- board outline added: 373.1 x 130.2 mm
Changed lines of the file:
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@@
   (general
     (thickness 1.6)
-    (drawings 588)
-    (tracks 605)
+    (drawings 600)
+    (tracks 612)
     (zones 0)
     (modules 201)
@@
     )
   )
+  (gr_line (start 110.33125 357.1875) (end 111.91875 357.1875) (layer Edge.Cuts) (width 0.05))
+  (gr_line (start 110.33125 244.475) (end 110.33125 357.1875) (layer Edge.Cuts) (width 0.05))
+  (gr_line (start 408.78125 357.21228) (end 111.91875 357.1875) (layer Edge.Cuts) (width 0.05))
+  (gr_line (start 483.39375 350.04375) (end 483.39375 357.1875) (layer Edge.Cuts) (width 0.05))
+  (gr_line (start 408.78125 357.21228) (end 483.39375 357.1875) (layer Edge.Cuts) (width 0.05))
+  (gr_line (start 483.39375 239.7125) (end 483.39375 350.04375) (layer Edge.Cuts) (width 0.05))
+  (gr_line (start 483.39375 227.0125) (end 481.0125 227.0125) (layer Edge.Cuts) (width 0.05))
+  (gr_line (start 483.39375 239.7125) (end 483.39375 227.0125) (layer Edge.Cuts) (width 0.05))
+  (gr_circle (center 408.78125 344.4875) (end 407.9875 357.1875) (layer Edge.Cuts) (width 0.05))
+  (gr_circle (center 470.69375 239.7125) (end 483.39375 239.7125) (layer Edge.Cuts) (width 0.05))
+  (gr_line (start 110.33125 227.0125) (end 481.0125 227.0125) (layer Edge.Cuts) (width 0.05))
+  (gr_line (start 110.33125 227.0125) (end 110.33125 244.475) (layer Edge.Cuts) (width 0.05))
   (gr_line (start 382.8755 337.34325) (end 396.8745 337.34325) (layer Dwgs.User) (width 0.2))
   (gr_line (start 401.9255 351.34272) (end 401.9255 337.34325) (layer Dwgs.User) (width 0.2))
@@
   (segment (start 210.34375 306.475) (end 220.54375 316.675) (width 0.254) (layer F.Cu) (net 111))
   (segment (start 210.34375 300.0375) (end 210.34375 306.475) (width 0.254) (layer F.Cu) (net 111))
+  (segment (start 219.23375 318.135) (end 219.23375 318.4525) (width 0.254) (layer F.Cu) (net 111))
+  (segment (start 219.23375 318.4525) (end 219.86875 319.0875) (width 0.254) (layer F.Cu) (net 111))
   (segment (start 219.23375 237.1725) (end 219.23375 237.49) (width 0.254) (layer F.Cu) (net 112))
   (segment (start 219.23375 237.49) (end 219.86875 238.125) (width 0.254) (layer F.Cu) (net 112))
@@
   (segment (start 238.91875 332.66875) (end 241.975 335.725) (width 0.254) (layer F.Cu) (net 112))
   (segment (start 238.91875 319.0875) (end 238.91875 332.66875) (width 0.254) (layer F.Cu) (net 112))
+  (segment (start 240.665 337.185) (end 240.665 337.5025) (width 0.254) (layer F.Cu) (net 112))
+  (segment (start 240.665 337.5025) (end 241.3 338.1375) (width 0.254) (layer F.Cu) (net 112))
+  (segment (start 241.3 338.1375) (end 241.3 341.3125) (width 0.254) (layer F.Cu) (net 112))
+  (segment (start 241.3 341.3125) (end 242.8875 342.9) (width 0.254) (layer F.Cu) (net 112))
+  (segment (start 242.8875 342.9) (end 251.61875 342.9) (width 0.254) (layer F.Cu) (net 112))
   (segment (start 238.28375 237.1725) (end 238.28375 237.49) (width 0.254) (layer F.Cu) (net 113))
   (segment (start 238.28375 237.49) (end 238.91875 238.125) (width 0.254) (layer F.Cu) (net 113))
