File: version 2 - STM32F303VC no RGB/GCS98v2.kicad_pcb (KiCad board)
At the start: 2 copper layers, 201 parts, among them SW1 SW_Push, SW2 SW_Push_SPDT, U1 STM32F303CCTx

Commit message: Revert "project corrupted"
This reverts commit 6e2c007335474fac45b2d4a7722601066718bb04.
Parts:
- D1, D10, D11, D12, D13, D14, D15, D16, D17, D18, D19, D2, D20, D21, D22, D23, D24, D25, D26, D27, D28, D29, D3, D30, D31, D32, D33, D34, D35, D36, D37, D38, D39, D4, D40, D41, D42, D43, D44, D45, D46, D47, D48, D49, D5, D50, D51, D52, D53, D54, D55, D56, D57, D58, D59, D6, D60, D61, D62, D63, D64, D65, D66, D67, D68, D69, D7, D70, D71, D72, D73, D74, D75, D76, D77, D78, D79, D8, D80, D81, D82, D83, D84, D85, D86, D87, D88, D89, D9, D90, D91, D92, D93, D94, D95, D96, D97, D98: moved to F.Cu
- moved SW2 254.3 mm to (73.4, 200.0)
- moved R1 254.3 mm to (80.4, 201.9)
- moved U1 254.3 mm to (63.0, 197.7)
- moved C1 248.3 mm to (59.5, 190.5)
- moved SW1 243.0 mm to (73.4, 193.2)
- moved D72 14.6 mm to (138.1, 325.5), turned to 90 degrees
- moved D67 14.0 mm to (381.0, 306.4), turned to 90 degrees
- moved D32 13.9 mm to (383.4, 268.4), turned to 90 degrees
- moved D10 12.4 mm to (302.4, 244.5), turned to 90 degrees
- moved D11 12.4 mm to (321.5, 244.5), turned to 90 degrees
- moved D12 12.4 mm to (340.5, 244.5), turned to 90 degrees
- moved D18 12.4 mm to (473.9, 244.5), turned to 90 degrees
- moved D20 12.4 mm to (145.3, 268.4), turned to 90 degrees
- moved D23 12.4 mm to (202.4, 268.4), turned to 90 degrees
- moved D26 12.4 mm to (259.6, 268.4), turned to 90 degrees
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Routing:
- net row1: track 349.0 -> 0.00 mm
- net row0: track 347.7 -> 0.00 mm
- net row3: track 341.9 -> 0.00 mm
- net row4: track 338.3 -> 0.00 mm
- net row2: track 325.2 -> 0.00 mm
- net row5: track 323.4 -> 0.00 mm
- net col11: track 120.6 -> 0.00 mm
- net col01: track 117.6 -> 0.00 mm
- net col10: track 117.5 -> 0.00 mm
- net col09: track 114.5 -> 0.00 mm
- net col02: track 114.0 -> 0.00 mm
- net col13: track 112.0 -> 0.00 mm
- net col00: track 110.0 -> 0.00 mm
- net col05: track 109.7 -> 0.00 mm
- net col14: track 101.6 -> 0.00 mm
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Other:
- net class Default: trace_width 0.254 -> 0.25
- net class Power removed
