File: GCSv1/GCS98v1.kicad_pcb (KiCad board)
At the start: 2 copper layers, 324 parts, among them J1 SM04B-SRSS-TB(LF)(SN), SW1 ESC, SW10 F9, SW11 F10, SW12 F11, SW13 F12, SW14 DEL, SW15 SW_MEC_5G, SW16 SW_MEC_5G, SW17 SW_MEC_5G, SW18 SW_MEC_5G, SW19 SW_MEC_5G, SW2 F1, SW20 SW_MEC_5G, SW21 SW_MEC_5G, SW22 SW_MEC_5G, SW23 SW_MEC_5G, SW24 SW_MEC_5G, SW25 SW_MEC_5G, SW26 SW_MEC_5G, SW27 SW_MEC_5G, SW28 SW_MEC_5G, SW29 SW_MEC_5G, SW3 F2, SW30 SW_MEC_5G, SW31 SW_MEC_5G, SW32 BKSPC, SW33 SW_MEC_5G, SW34 SW_MEC_5G, SW35 SW_MEC_5G, SW36 SW_MEC_5G, SW37 TAB, SW38 SW_MEC_5G, SW39 SW_MEC_5G, SW4 F3, SW40 SW_MEC_5G, SW41 SW_MEC_5G, SW42 SW_MEC_5G, SW43 SW_MEC_5G, SW44 SW_MEC_5G, SW45 SW_MEC_5G, SW46 SW_MEC_5G, SW47 SW_MEC_5G, SW48 SW_MEC_5G, SW49 SW_MEC_5G, SW5 F4, SW50 BSLSH, SW51 SW_MEC_5G, SW52 SW_MEC_5G, SW53 SW_MEC_5G, SW54 SW_MEC_5G, SW55 CAPS, SW56 SW_MEC_5G, SW57 SW_MEC_5G, SW58 SW_MEC_5G, SW59 SW_MEC_5G, SW6 F5, SW60 SW_MEC_5G, SW61 SW_MEC_5G, SW62 SW_MEC_5G, SW63 SW_MEC_5G, SW64 SW_MEC_5G, SW65 SW_MEC_5G, SW66 SW_MEC_5G, SW67 ENTER, SW68 SW_MEC_5G, SW69 SW_MEC_5G, SW7 F6, SW70 SW_MEC_5G, SW71 SW_MEC_5G, SW72 LSHFT, SW73 SW_MEC_5G, SW74 SW_MEC_5G, SW75 SW_MEC_5G, SW76 SW_MEC_5G, SW77 SW_MEC_5G, SW78 SW_MEC_5G, SW79 SW_MEC_5G, SW8 F7, SW80 SW_MEC_5G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

Commit message: pick-and-place simulator
Parts:
- SW15: value SW_MEC_5G -> F13
- SW16: value SW_MEC_5G -> F14
- SW17: value SW_MEC_5G -> F15
- SW18: value SW_MEC_5G -> F16
- SW19: value SW_MEC_5G -> TILDE
- SW20: value SW_MEC_5G -> 1
- SW21: value SW_MEC_5G -> 2
- SW22: value SW_MEC_5G -> 3
- SW23: value SW_MEC_5G -> 4
- SW24: value SW_MEC_5G -> 5
- SW25: value SW_MEC_5G -> 6
- SW26: value SW_MEC_5G -> 7
- SW27: value SW_MEC_5G -> 8
- SW28: value SW_MEC_5G -> 9
- SW29: value SW_MEC_5G -> 0
- SW30: value SW_MEC_5G -> DASH
- SW31: value SW_MEC_5G -> EQUAL
- SW33: value SW_MEC_5G -> MOP1
- SW34: value SW_MEC_5G -> MOP2
- SW35: value SW_MEC_5G -> MOP3
- SW36: value SW_MEC_5G -> MOP4
- moved SW35 430.4 mm to (473.9, 277.8)
- moved SW33 385.1 mm to (435.8, 277.8)
- moved SW16 297.7 mm to (454.8, 254.0)
- moved SW28 181.7 mm to (316.7, 277.8)
- moved SW22 164.3 mm to (202.4, 277.8)
- moved SW25 139.8 mm to (259.6, 277.8)
- moved SW20 103.6 mm to (164.3, 277.8)
- moved SW19 82.8 mm to (145.3, 277.8)
Changed lines of the file:
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@@
       (effects (font (size 1 1) (thickness 0.15)))
     )
-    (fp_text value SW_MEC_5G (at 0 -7.9375) (layer Dwgs.User)
+    (fp_text value MOP4 (at 0 -7.9375) (layer Dwgs.User)
       (effects (font (size 1 1) (thickness 0.15)))
     )
@@
   )
   (module MX_Alps_Hybrid:MX-1U-NoLED (layer F.Cu)
-    (at 93.94375 75.4725)
+    (at 473.86875 277.8125)
     (fp_text reference SW35 (at 0 3.175) (layer Dwgs.User)
       (effects (font (size 1 1) (thickness 0.15)))
     )
-    (fp_text value SW_MEC_5G (at 0 -7.9375) (layer Dwgs.User)
+    (fp_text value MOP3 (at 0 -7.9375) (layer Dwgs.User)
       (effects (font (size 1 1) (thickness 0.15)))
     )
@@
       (effects (font (size 1 1) (thickness 0.15)))
     )
-    (fp_text value SW_MEC_5G (at 0 -7.9375) (layer Dwgs.User)
+    (fp_text value MOP2 (at 0 -7.9375) (layer Dwgs.User)
       (effects (font (size 1 1) (thickness 0.15)))
     )
@@
   )
   (module MX_Alps_Hybrid:MX-1U-NoLED (layer F.Cu)
-    (at 70.13375 156.9125)
+    (at 435.76875 277.8125)
     (fp_text reference SW33 (at 0 3.175) (layer Dwgs.User)
       (effects (font (size 1 1) (thickness 0.15)))
     )
-    (fp_text value SW_MEC_5G (at 0 -7.9375) (layer Dwgs.User)
+    (fp_text value MOP1 (at 0 -7.9375) (layer Dwgs.User)
       (effects (font (size 1 1) (thickness 0.15)))
     )
@@
       (effects (font (size 1 1) (thickness 0.15)))
     )
-    (fp_text value SW_MEC_5G (at 0 -7.9375) (layer Dwgs.User)
+    (fp_text value EQUAL (at 0 -7.9375) (layer Dwgs.User)
       (effects (font (size 1 1) (thickness 0.15)))
     )
@@
       (effects (font (size 1 1) (thickness 0.15)))
     )
-    (fp_text value SW_MEC_5G (at 0 -7.9375) (layer Dwgs.User)
+    (fp_text value DASH (at 0 -7.9375) (layer Dwgs.User)
       (effects (font (size 1 1) (thickness 0.15)))
     )
@@
       (effects (font (size 1 1) (thickness 0.15)))
     )
-    (fp_text value SW_MEC_5G (at 0 -7.9375) (layer Dwgs.User)
+    (fp_text value 0 (at 0 -7.9375) (layer Dwgs.User)
       (effects (font (size 1 1) (thickness 0.15)))
     )
@@
   )
   (module MX_Alps_Hybrid:MX-1U-NoLED (layer F.Cu)
-    (at 166.37375 175.8325)
+    (at 316.70625 277.8125)
     (fp_text reference SW28 (at 0 3.175) (layer Dwgs.User)
       (effects (font (size 1 1) (thickness 0.15)))
     )
-    (fp_text value SW_MEC_5G (at 0 -7.9375) (layer Dwgs.User)
+    (fp_text value 9 (at 0 -7.9375) (layer Dwgs.User)
       (effects (font (size 1 1) (thickness 0.15)))
     )
@@
       (effects (font (size 1 1) (thickness 0.15)))
     )
-    (fp_text value SW_MEC_5G (at 0 -7.9375) (layer Dwgs.User)
+    (fp_text value 8 (at 0 -7.9375) (layer Dwgs.User)
       (effects (font (size 1 1) (thickness 0.15)))
     )
@@
       (effects (font (size 1 1) (thickness 0.15)))
     )
-    (fp_text value SW_MEC_5G (at 0 -7.9375) (layer Dwgs.User)
+    (fp_text value 7 (at 0 -7.9375) (layer Dwgs.User)
       (effects (font (size 1 1) (thickness 0.15)))
     )
@@
   )
   (module MX_Alps_Hybrid:MX-1U-NoLED (layer F.Cu)
-    (at 146.17375 196.0325)
+    (at 259.55625 277.8125)
     (fp_text reference SW25 (at 0 3.175) (layer Dwgs.User)
       (effects (font (size 1 1) (thickness 0.15)))
     )
-    (fp_text value SW_MEC_5G (at 0 -7.9375) (layer Dwgs.User)
+    (fp_text value 6 (at 0 -7.9375) (layer Dwgs.User)
       (effects (font (size 1 1) (thickness 0.15)))
     )
@@
       (effects (font (size 1 1) (thickness 0.15)))
     )
-    (fp_text value SW_MEC_5G (at 0 -7.9375) (layer Dwgs.User)
+    (fp_text value 5 (at 0 -7.9375) (layer Dwgs.User)
       (effects (font (size 1 1) (thickness 0.15)))
     )
@@
       (effects (font (size 1 1) (thickness 0.15)))
     )
-    (fp_text value SW_MEC_5G (at 0 -7.9375) (layer Dwgs.User)
+    (fp_text value 4 (at 0 -7.9375) (layer Dwgs.User)
       (effects (font (size 1 1) (thickness 0.15)))
     )
@@
   )
   (module MX_Alps_Hybrid:MX-1U-NoLED (layer F.Cu)
-    (at 221.05375 114.5925)
+    (at 202.40625 277.8125)
     (fp_text reference SW22 (at 0 3.175) (layer Dwgs.User)
       (effects (font (size 1 1) (thickness 0.15)))
     )
-    (fp_text value SW_MEC_5G (at 0 -7.9375) (layer Dwgs.User)
+    (fp_text value 3 (at 0 -7.9375) (layer Dwgs.User)
       (effects (font (size 1 1) (thickness 0.15)))
     )
@@
       (effects (font (size 1 1) (thickness 0.15)))
     )
-    (fp_text value SW_MEC_5G (at 0 -7.9375) (layer Dwgs.User)
+    (fp_text value 2 (at 0 -7.9375) (layer Dwgs.User)
       (effects (font (size 1 1) (thickness 0.15)))
     )
@@
   )
   (module MX_Alps_Hybrid:MX-1U-NoLED (layer F.Cu)
-    (at 146.17375 175.8325)
+    (at 164.30625 277.8125)
     (fp_text reference SW20 (at 0 3.175) (layer Dwgs.User)
       (effects (font (size 1 1) (thickness 0.15)))
     )
-    (fp_text value SW_MEC_5G (at 0 -7.9375) (layer Dwgs.User)
+    (fp_text value 1 (at 0 -7.9375) (layer Dwgs.User)
       (effects (font (size 1 1) (thickness 0.15)))
     )
@@
   )
   (module MX_Alps_Hybrid:MX-1U-NoLED (layer F.Cu)
-    (at 125.97375 197.3125)
+    (at 145.25625 277.8125)
     (fp_text reference SW19 (at 0 3.175) (layer Dwgs.User)
       (effects (font (size 1 1) (thickness 0.15)))
     )
-    (fp_text value SW_MEC_5G (at 0 -7.9375) (layer Dwgs.User)
+    (fp_text value TILDE (at 0 -7.9375) (layer Dwgs.User)
       (effects (font (size 1 1) (thickness 0.15)))
     )
@@
       (effects (font (size 1 1) (thickness 0.15)))
     )
-    (fp_text value SW_MEC_5G (at 0 -7.9375) (layer Dwgs.User)
+    (fp_text value F16 (at 0 -7.9375) (layer Dwgs.User)
       (effects (font (size 1 1) (thickness 0.15)))
     )
@@
       (effects (font (size 1 1) (thickness 0.15)))
     )
-    (fp_text value SW_MEC_5G (at 0 -7.9375) (layer Dwgs.User)
+    (fp_text value F15 (at 0 -7.9375) (layer Dwgs.User)
       (effects (font (size 1 1) (thickness 0.15)))
     )
@@
   )
   (module MX_Alps_Hybrid:MX-1U-NoLED (layer F.Cu)
-    (at 254.55375 33.7925)
+    (at 454.81875 254)
     (fp_text reference SW16 (at 0 3.175) (layer Dwgs.User)
       (effects (font (size 1 1) (thickness 0.15)))
     )
-    (fp_text value SW_MEC_5G (at 0 -7.9375) (layer Dwgs.User)
+    (fp_text value F14 (at 0 -7.9375) (layer Dwgs.User)
       (effects (font (size 1 1) (thickness 0.15)))
     )
@@
       (effects (font (size 1 1) (thickness 0.15)))
     )
-    (fp_text value SW_MEC_5G (at 0 -7.9375) (layer Dwgs.User)
-      (effects (font (size 1 1) (thickness 0.15)))
-    )
+    (fp_text value F13 (at 0 -7.9375) (layer Dwgs.User)
+      (effects (font (size 1 1) (thickness 0.15)))
+    )

Commit message: finished placing switches
Parts:
- SW38: value SW_MEC_5G -> Q
- SW39: value SW_MEC_5G -> W
- SW40: value SW_MEC_5G -> E
- SW41: value SW_MEC_5G -> R
- SW42: value SW_MEC_5G -> T
- SW43: value SW_MEC_5G -> Y
- SW44: value SW_MEC_5G -> U
- SW45: value SW_MEC_5G -> I
- SW46: value SW_MEC_5G -> O
- SW47: value SW_MEC_5G -> P
- SW48: value SW_MEC_5G -> LBRKT
- SW49: value SW_MEC_5G -> RBRKT
- SW51: value SW_MEC_5G -> NUM7
- SW52: value SW_MEC_5G -> NUM8
- SW53: value SW_MEC_5G -> NUM9
- SW54: value SW_MEC_5G -> MOP5
- SW56: value SW_MEC_5G -> A
- SW57: value SW_MEC_5G -> S
- SW58: value SW_MEC_5G -> D
- SW59: value SW_MEC_5G -> F
- SW60: value SW_MEC_5G -> G
- SW61: value SW_MEC_5G -> H
- SW62: value SW_MEC_5G -> J
- SW63: value SW_MEC_5G -> K
- SW64: value SW_MEC_5G -> L
- SW65: value SW_MEC_5G -> SMCLN
- SW66: value SW_MEC_5G -> APOST
- SW68: value SW_MEC_5G -> NUM4
- SW69: value SW_MEC_5G -> NUM5
- SW70: value SW_MEC_5G -> NUM6
- SW71: value SW_MEC_5G -> MOP6
- SW73: value SW_MEC_5G -> Z
- SW74: value SW_MEC_5G -> X
- SW75: value SW_MEC_5G -> C
- SW76: value SW_MEC_5G -> V
- SW77: value SW_MEC_5G -> B
- SW78: value SW_MEC_5G -> N
- SW79: value SW_MEC_5G -> M
- SW80: value SW_MEC_5G -> COMMA
- SW81: value SW_MEC_5G -> PRD
- SW82: value SW_MEC_5G -> SLSH
- SW84: value SW_MEC_5G -> UP
- SW85: value SW_MEC_5G -> NUM1
- SW86: value SW_MEC_5G -> NUM2
- SW87: value SW_MEC_5G -> NUM3
- SW95: value SW_MEC_5G -> LEFT
- SW96: value SW_MEC_5G -> DOWN
- SW97: value SW_MEC_5G -> RIGHT
- moved C10 527.7 mm to (546.2, 101.3)
- moved C11 527.7 mm to (554.0, 91.5)
- moved C12 527.7 mm to (546.2, 104.3)
- moved C15 527.7 mm to (541.4, 98.3)
- moved C16 527.7 mm to (558.9, 94.5)
- moved C7 527.7 mm to (558.9, 91.5)
- moved C8 527.7 mm to (551.0, 97.5)
- moved C9 527.7 mm to (554.0, 94.5)
- moved D197 527.7 mm to (555.5, 106.5)
- moved D198 527.7 mm to (559.8, 106.4)
- moved J1 527.7 mm to (542.9, 96.1)
- moved R4 527.7 mm to (551.0, 106.5)
- moved SW99 527.7 mm to (532.4, 104.7)
- moved Y1 527.7 mm to (540.5, 104.2)
- moved C13 527.7 mm to (546.2, 98.3)
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
Commit message: tmp commit to revert
Other:
- board outline added: 376.2 x 133.3 mm
Changed lines of the file:
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@@
   (general
     (thickness 1.6)
-    (drawings 584)
+    (drawings 592)
     (tracks 0)
     (zones 0)
@@
     )
   )
+  (gr_line (start 507.20625 239.7125) (end 130.96875 239.7125) (layer Edge.Cuts) (width 0.05))
+  (gr_line (start 507.20625 368.3) (end 507.20625 239.7125) (layer Edge.Cuts) (width 0.05))
+  (gr_line (start 445.29375 368.3) (end 507.20625 368.3) (layer Edge.Cuts) (width 0.05))
+  (gr_line (start 445.29375 373.0625) (end 445.29375 368.3) (layer Edge.Cuts) (width 0.05))
+  (gr_line (start 326.23125 373.0625) (end 445.29375 373.0625) (layer Edge.Cuts) (width 0.05))
+  (gr_line (start 326.23125 368.3) (end 326.23125 373.0625) (layer Edge.Cuts) (width 0.05))
+  (gr_line (start 130.96875 368.3) (end 326.23125 368.3) (layer Edge.Cuts) (width 0.05))
+  (gr_line (start 130.96875 239.7125) (end 130.96875 368.3) (layer Edge.Cuts) (width 0.05))
   (gr_line (start 373.644 351.74288) (end 373.644 365.74235) (layer Cmts.User) (width 0.2))
   (gr_line (start 335.831 351.74288) (end 349.832 351.74288) (layer Cmts.User) (width 0.2))

Commit message: i think i get my edge cuts back?
all the revert commits I have done thus far is because layout editor crashes, and Event Viewer pointed to "NVIDIA OpenGL Driver" in each instance, and then both schematic and layout editors would crash when launching. Went to NVIDIA website to install the driver, selecting the option to perform a clean install in the wizard.

PSA: the express installation option in the driver installer and GeForce Experience leave a lot of duplicate files for programs to find and incorrectly use, make sure to perform a clean install every time you update NVIDIA drivers
Other:
- board outline removed
Changed lines of the file:
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@@
   (general
     (thickness 1.6)
-    (drawings 592)
+    (drawings 584)
     (tracks 0)
     (zones 0)
@@
     )
   )
-  (gr_line (start 507.20625 239.7125) (end 130.96875 239.7125) (layer Edge.Cuts) (width 0.05))
-  (gr_line (start 507.20625 368.3) (end 507.20625 239.7125) (layer Edge.Cuts) (width 0.05))
-  (gr_line (start 445.29375 368.3) (end 507.20625 368.3) (layer Edge.Cuts) (width 0.05))
-  (gr_line (start 445.29375 373.0625) (end 445.29375 368.3) (layer Edge.Cuts) (width 0.05))
-  (gr_line (start 326.23125 373.0625) (end 445.29375 373.0625) (layer Edge.Cuts) (width 0.05))
-  (gr_line (start 326.23125 368.3) (end 326.23125 373.0625) (layer Edge.Cuts) (width 0.05))
-  (gr_line (start 130.96875 368.3) (end 326.23125 368.3) (layer Edge.Cuts) (width 0.05))
-  (gr_line (start 130.96875 239.7125) (end 130.96875 368.3) (layer Edge.Cuts) (width 0.05))
   (gr_line (start 373.644 351.74288) (end 373.644 365.74235) (layer Cmts.User) (width 0.2))
   (gr_line (start 335.831 351.74288) (end 349.832 351.74288) (layer Cmts.User) (width 0.2))

Commit message: RGB edition pick and place machine by Corsair
Parts:
- C1, C10, C11, C12, C13, C14, C15, C16, C17, C18, C2, C3, C4, C5, C6, C7, C8, C9, D1, D10, D100, D101, D102, D103, D104, D105, D106, D107, D108, D109, D11, D110, D111, D112, D113, D114, D115, D116, D117, D118, D119, D12, D120, D121, D122, D123, D124, D125, D126, D127, D128, D129, D13, D130, D131, D132, D133, D134, D135, D136, D137, D138, D139, D14, D140, D141, D142, D143, D144, D145, D146, D147, D148, D149, D15, D150, D151, D152, D153, D154, D155, D156, D157, D158, D159, D16, D160, D161, D162, D163, D164, D165, D166, D167, D168, D169, D17, D170, D171, D172, D173, D174, D175, D177, D178, D179, D18, D180, D181, D182, D183, D184, D185, D186, D187, D188, D189, D19, D190, D191, D192, D193, D194, D195, D196, D197, D198, D2, D20, D21, D22, D23, D24, D25, D26, D27, D28, D29, D3, D30, D31, D32, D33, D34, D35, D36, D37, D38, D39, D4, D40, D41, D42, D43, D44, D45, D46, D47, D48, D49, D5, D50, D51, D52, D53, D54, D55, D56, D57, D58, D59, D6, D60, D61, D62, D63, D64, D65, D66, D67, D68, D69, D7, D70, D71, D72, D73, D74, D75, D76, D77, D78, D79, D8, D80, D81, D82, D83, D84, D85, D86, D87, D88, D89, D9, D90, D91, D92, D93, D94, D95, D96, D97, D98, D99, J1, R1, R2, R3, R4, R5, SW99, U1, U2, Y1: moved to B.Cu
- moved D177 451.8 mm to (147.6, 359.6)
- moved D124 441.6 mm to (473.9, 321.5)
- moved D178 425.7 mm to (171.4, 359.6)
- moved D143 414.8 mm to (157.2, 340.5)
- moved D37 398.0 mm to (145.3, 283.4)
- moved D74 388.4 mm to (173.8, 302.4)
- moved D39 363.7 mm to (183.4, 283.4)
- moved D146 343.1 mm to (226.2, 340.5)
- moved D2 331.6 mm to (169.1, 259.6)
- moved D144 328.7 mm to (188.1, 340.5)
- moved D78 325.2 mm to (250.0, 302.4)
- moved D186 321.5 mm to (464.3, 359.6)
- moved D79 320.2 mm to (269.1, 302.4)
- moved D183 309.5 mm to (392.9, 364.3)
- moved D179 306.1 mm to (195.3, 359.6)
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Other:
- board outline added: 376.2 x 133.3 mm

Commit message: matrix pick and place done, now to routing it
Parts:
- D176: moved to B.Cu
- moved D36 348.9 mm to (498.5, 247.7), turned to 270 degrees
- moved D70 292.3 mm to (460.4, 271.5), turned to 270 degrees
- moved D196 288.5 mm to (469.9, 347.7), turned to 270 degrees
- moved D35 277.4 mm to (479.4, 247.7), turned to 270 degrees
- moved D71 274.3 mm to (479.4, 271.5), turned to 270 degrees
- moved D187 270.9 mm to (153.2, 347.7), turned to 270 degrees
- moved D72 267.1 mm to (498.5, 271.5), turned to 270 degrees
- moved D188 245.5 mm to (177.0, 347.7), turned to 270 degrees
- moved D194 244.2 mm to (417.5, 352.4), turned to 270 degrees
- moved R1 239.2 mm to (517.5, 170.7)
- moved D189 233.1 mm to (200.8, 347.7), turned to 270 degrees
- moved D91 230.3 mm to (155.6, 290.5), turned to 270 degrees
- moved D126 221.1 mm to (158.0, 309.6), turned to 270 degrees
- moved D169 215.5 mm to (346.1, 328.6), turned to 270 degrees
- moved D195 204.1 mm to (436.6, 352.4), turned to 270 degrees
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
Commit message: backup before changing symbols
realized the switch symbol I had been using actually has 4 pins, in two stacks of two (really fucking dumb)
Parts:
- moved C1 331.2 mm to (258.0, 389.7)
- moved C10 331.2 mm to (297.8, 384.4)
- moved C12 331.2 mm to (297.8, 381.4)
- moved C15 331.2 mm to (292.9, 387.5)
- moved C16 331.2 mm to (310.4, 391.2)
- moved C3 331.2 mm to (258.0, 377.7)
- moved C4 331.2 mm to (258.0, 380.7)
- moved C5 331.2 mm to (258.0, 383.7)
- moved C6 331.2 mm to (258.0, 386.7)
- moved C7 331.2 mm to (310.4, 394.3)
- moved C8 331.2 mm to (302.6, 388.2)
- moved D197 331.2 mm to (307.1, 379.2)
- moved D198 331.2 mm to (311.3, 379.4)
- moved J1 331.2 mm to (294.4, 389.7)
- moved R4 331.2 mm to (302.6, 379.2)
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Routing:
- net row1: track 0.00 -> 352.3 mm
- net row0: track 0.00 -> 348.5 mm
- net row3: track 0.00 -> 344.8 mm
- net row2: track 0.00 -> 343.2 mm
- net row4: track 0.00 -> 339.0 mm
- net row5: track 0.00 -> 323.3 mm
- net Net-(D176-Pad2): track 0.00 -> 20.7 mm
- net Net-(D161-Pad2): track 0.00 -> 3.74 mm
- net Net-(D142-Pad2): track 0.00 -> 3.40 mm
- net Net-(D136-Pad2): track 0.00 -> 3.40 mm
- net Net-(D131-Pad2): track 0.00 -> 3.40 mm
- net Net-(D135-Pad2): track 0.00 -> 3.40 mm
- net Net-(D130-Pad2): track 0.00 -> 3.40 mm
- net Net-(D126-Pad2): track 0.00 -> 3.40 mm
- net Net-(D129-Pad2): track 0.00 -> 3.40 mm
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
Commit message: another backup before changing rgb symbol
Parts:
- moved J1 37.4 mm to (297.7, 352.4), turned to 315 degrees
- moved U1 24.9 mm to (296.9, 368.3), turned to 45 degrees
Connections:
- SW1 pad 1: Net-(D19-Pad2) -> col00
- SW10 pad 1: Net-(D28-Pad2) -> col09
- SW11 pad 1: Net-(D29-Pad2) -> col10
- SW12 pad 1: Net-(D30-Pad2) -> col11
- SW13 pad 1: Net-(D31-Pad2) -> col12
- SW14 pad 1: Net-(D32-Pad2) -> col13
- SW15 pad 1: Net-(D33-Pad2) -> col14
- SW16 pad 1: Net-(D34-Pad2) -> col15
- SW17 pad 1: Net-(D35-Pad2) -> col16
- SW18 pad 1: Net-(D36-Pad2) -> col17
- SW19 pad 1: Net-(D55-Pad2) -> col00
- SW2 pad 1: Net-(D20-Pad2) -> col01
- SW20 pad 1: Net-(D56-Pad2) -> col01
- SW21 pad 1: Net-(D57-Pad2) -> col02
- SW22 pad 1: Net-(D58-Pad2) -> col03
- SW23 pad 1: Net-(D59-Pad2) -> col04
- SW24 pad 1: Net-(D60-Pad2) -> col05
- SW25 pad 1: Net-(D61-Pad2) -> col06
- SW26 pad 1: Net-(D62-Pad2) -> col07
- SW27 pad 1: Net-(D63-Pad2) -> col08
- SW28 pad 1: Net-(D64-Pad2) -> col09
- SW29 pad 1: Net-(D65-Pad2) -> col10
- SW3 pad 1: Net-(D21-Pad2) -> col02
- SW30 pad 1: Net-(D66-Pad2) -> col11
- SW31 pad 1: Net-(D67-Pad2) -> col12
- SW32 pad 1: Net-(D68-Pad2) -> col13
- SW33 pad 1: Net-(D69-Pad2) -> col14
- SW34 pad 1: Net-(D70-Pad2) -> col15
- SW35 pad 1: Net-(D71-Pad2) -> col16
- SW36 pad 1: Net-(D72-Pad2) -> col17
- SW37 pad 1: Net-(D91-Pad2) -> col00
- SW38 pad 1: Net-(D92-Pad2) -> col01
- SW39 pad 1: Net-(D93-Pad2) -> col02
- SW4 pad 1: Net-(D22-Pad2) -> col03
- SW40 pad 1: Net-(D94-Pad2) -> col03
- SW41 pad 1: Net-(D95-Pad2) -> col04
- SW42 pad 1: Net-(D96-Pad2) -> col05
- SW43 pad 1: Net-(D97-Pad2) -> col06
- SW44 pad 1: Net-(D98-Pad2) -> col07
- SW45 pad 1: Net-(D99-Pad2) -> col08
- SW46 pad 1: Net-(D100-Pad2) -> col09
- SW47 pad 1: Net-(D101-Pad2) -> col10
- SW48 pad 1: Net-(D102-Pad2) -> col11
- SW49 pad 1: Net-(D103-Pad2) -> col12
- SW5 pad 1: Net-(D23-Pad2) -> col04
- SW50 pad 1: Net-(D104-Pad2) -> col13
- SW51 pad 1: Net-(D105-Pad2) -> col14
- SW52 pad 1: Net-(D106-Pad2) -> col15
- SW53 pad 1: Net-(D107-Pad2) -> col16
- SW54 pad 1: Net-(D108-Pad2) -> col17
- SW55 pad 1: Net-(D126-Pad2) -> col00
- SW56 pad 1: Net-(D127-Pad2) -> col01
- SW57 pad 1: Net-(D128-Pad2) -> col02
- SW58 pad 1: Net-(D129-Pad2) -> col03
- SW59 pad 1: Net-(D130-Pad2) -> col04
- SW6 pad 1: Net-(D24-Pad2) -> col05
- SW60 pad 1: Net-(D131-Pad2) -> col05
- SW61 pad 1: Net-(D132-Pad2) -> col06
- SW62 pad 1: Net-(D133-Pad2) -> col07
- SW63 pad 1: Net-(D134-Pad2) -> col08
- SW64 pad 1: Net-(D135-Pad2) -> col09
- SW65 pad 1: Net-(D136-Pad2) -> col10
- SW66 pad 1: Net-(D137-Pad2) -> col11
- SW67 pad 1: Net-(D138-Pad2) -> col13
- SW68 pad 1: Net-(D139-Pad2) -> col14
- SW69 pad 1: Net-(D140-Pad2) -> col15
- SW7 pad 1: Net-(D25-Pad2) -> col06
- SW70 pad 1: Net-(D141-Pad2) -> col16
- SW71 pad 1: Net-(D142-Pad2) -> col17
- SW72 pad 1: Net-(D160-Pad2) -> col00
- SW73 pad 1: Net-(D161-Pad2) -> col01
- SW74 pad 1: Net-(D162-Pad2) -> col02
- SW75 pad 1: Net-(D163-Pad2) -> col03
- SW76 pad 1: Net-(D164-Pad2) -> col04
- SW77 pad 1: Net-(D165-Pad2) -> col05
- SW78 pad 1: Net-(D166-Pad2) -> col06
- SW79 pad 1: Net-(D167-Pad2) -> col07
- SW8 pad 1: Net-(D26-Pad2) -> col07
- SW80 pad 1: Net-(D168-Pad2) -> col08
- SW81 pad 1: Net-(D169-Pad2) -> col09
- SW82 pad 1: Net-(D170-Pad2) -> col10
- SW83 pad 1: Net-(D171-Pad2) -> col11
- SW84 pad 1: Net-(D172-Pad2) -> col13
- SW85 pad 1: Net-(D173-Pad2) -> col14
- SW86 pad 1: Net-(D174-Pad2) -> col15
- SW87 pad 1: Net-(D175-Pad2) -> col16
- SW88 pad 1: Net-(D176-Pad2) -> col17
- SW89 pad 1: Net-(D187-Pad2) -> col00
- SW9 pad 1: Net-(D27-Pad2) -> col08
- SW90 pad 1: Net-(D188-Pad2) -> col01
- SW91 pad 1: Net-(D189-Pad2) -> col02
- SW92 pad 1: Net-(D190-Pad2) -> col05
- SW93 pad 1: Net-(D191-Pad2) -> col09
- SW94 pad 1: Net-(D192-Pad2) -> col10
- SW95 pad 1: Net-(D193-Pad2) -> col11
- SW96 pad 1: Net-(D194-Pad2) -> col13
- SW97 pad 1: Net-(D195-Pad2) -> col14
- SW98 pad 1: Net-(D196-Pad2) -> col16
Routing:
- net col11: track 0.00 -> 122.1 mm
- net col10: track 0.00 -> 119.6 mm
- net col09: track 0.00 -> 117.6 mm
- net col01: track 0.00 -> 115.2 mm
- net col13: track 0.00 -> 114.6 mm
- net col05: track 0.00 -> 112.8 mm
- net col02: track 0.00 -> 112.3 mm
- net col00: track 0.00 -> 107.2 mm
- net col14: track 0.00 -> 104.7 mm
- net col16: track 0.00 -> 104.0 mm
- net col03: track 0.00 -> 92.8 mm
- net col17: track 0.00 -> 92.1 mm
- net col06: track 0.00 -> 90.8 mm
- net col08: track 0.00 -> 90.8 mm
- net col04: track 0.00 -> 90.8 mm
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