File: GCSv1/GCS98v1.kicad_pcb (KiCad board)
At the start: 2 copper layers, 376.2 x 133.3 mm, 324 parts, among them J1 SM04B-SRSS-TB(LF)(SN), SW1 ESC, SW10 F9, SW11 F10, SW12 F11, SW13 F12, SW14 DEL, SW15 F13, SW16 F14, SW17 F15, SW18 F16, SW19 TILDE, SW2 F1, SW20 1, SW21 2, SW22 3, SW23 4, SW24 5, SW25 6, SW26 7, SW27 8, SW28 9, SW29 0, SW3 F2, SW30 DASH, SW31 EQUAL, SW32 BKSPC, SW33 MOP1, SW34 MOP2, SW35 MOP3, SW36 MOP4, SW37 TAB, SW38 Q, SW39 W, SW4 F3, SW40 E, SW41 R, SW42 T, SW43 Y, SW44 U, SW45 I, SW46 O, SW47 P, SW48 LBRKT, SW49 RBRKT, SW5 F4, SW50 BSLSH, SW51 NUM7, SW52 NUM8, SW53 NUM9, SW54 MOP5, SW55 CAPS, SW56 A, SW57 S, SW58 D, SW59 F, SW6 F5, SW60 G, SW61 H, SW62 J, SW63 K, SW64 L, SW65 SMCLN, SW66 APOST, SW67 ENTER, SW68 NUM4, SW69 NUM5, SW7 F6, SW70 NUM6, SW71 MOP6, SW72 LSHFT, SW73 Z, SW74 X, SW75 C, SW76 V, SW77 B, SW78 N, SW79 M, SW8 F7, SW80 COMMA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

Commit message: matrix wiring 90% done
still need to figure out how to get power to LEDs (probably route 5V through top plane, then fill in the rest of the top with ground; not much point to filling bottom plane with ground considering all the routing for rows, LED's, and other circuitry under the spacebar)

also need to get rows and columns into buses in the spacebar area, otherwise all that's left is min-maxing the positions of connector, MCU, VRM, resonator, and capacitors/resistors/diodes
Parts:
- D1, D10, D109, D11, D110, D111, D112, D113, D114, D115, D116, D117, D118, D119, D12, D120, D121, D122, D123, D124, D125, D13, D14, D143, D144, D145, D146, D147, D148, D149, D15, D150, D151, D152, D153, D154, D155, D156, D157, D158, D159, D16, D17, D177, D178, D179, D18, D180, D181, D182, D183, D184, D185, D186, D2, D3, D37, D38, D39, D4, D40, D41, D42, D43, D44, D45, D46, D47, D48, D49, D5, D50, D51, D52, D53, D54, D6, D7, D73, D74, D75, D76, D77, D78, D79, D8, D80, D81, D82, D83, D84, D85, D86, D87, D88, D89, D9, D90: footprint acheron_Components:SK6812MINI_3535_6028_3.2x2.8mm_Round -> custom symbols and footprints:SK6812MINI_3535_6028_3.2x2.8mm_Round_ROTATED
- moved J1 62.0 mm to (347.9, 388.7)
- moved U1 50.5 mm to (337.3, 398.5)
- moved R1 46.5 mm to (231.8, 361.9), turned to 180 degrees
- moved D196 5.56 mm to (464.3, 347.4)
- moved D108 5.56 mm to (492.9, 290.5)
- moved D142 5.56 mm to (492.9, 309.6)
- moved D36 5.56 mm to (492.9, 247.7)
- moved D72 5.56 mm to (492.9, 271.5)
- moved D176 5.12 mm to (492.9, 333.1)
Connections:
- net LED renamed LED_IN
Routing:
- net Net-(D109-Pad4): track 0.00 -> 378.6 mm
- net Net-(D1-Pad4): track 0.00 -> 374.6 mm
- net Net-(D37-Pad4): track 0.00 -> 370.7 mm
- net Net-(D125-Pad2): track 0.00 -> 365.4 mm
- net Net-(D143-Pad4): track 0.00 -> 335.1 mm
- net Net-(D177-Pad4): track 0.00 -> 88.4 mm
- net Net-(D180-Pad2): track 0.00 -> 82.4 mm
- net Net-(D179-Pad2): track 0.00 -> 66.8 mm
- net Net-(D121-Pad2): track 0.00 -> 31.1 mm
- net Net-(D185-Pad2): track 0.00 -> 29.4 mm
- net Net-(D50-Pad2): track 0.00 -> 28.7 mm
- net Net-(D120-Pad2): track 0.00 -> 26.3 mm
- net Net-(D143-Pad2): track 0.00 -> 26.3 mm
- net Net-(D154-Pad2): track 0.00 -> 25.9 mm
- net Net-(D86-Pad2): track 0.00 -> 24.0 mm
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
Commit message: redid matrix routing, not doing USB daughter board because of parts availability
Parts:
- removed D100, D101, D102, D103, D104, D105, D106, D107, D108, D126, D127, D128, D129, D130, D131, D132, D133, D134, D135, D136, D137, D138, D139, D140, D141, D142, D160, D161, D162, D163, D164, D165, D166, D167, D168, D169, D170, D171, D172, D173, D174, D175, D176, D187, D188, D189, D190, D191, D192, D193, D194, D195, D196: D, Diode_SMD:D_0805_2012Metric_Pad1.15x1.40mm_HandSolder
- removed D109, D110, D111, D112, D113, D114, D115, D116, D117, D118, D119, D120, D121, D122, D123, D124, D125, D143, D144, D145, D146, D147, D148, D149, D150, D151, D152, D153, D154, D155, D156, D157, D158, D159, D177, D178, D179, D180, D181, D182, D183, D184, D185, D186: SK6812MINI-E, custom symbols and footprints:SK6812MINI_3535_6028_3.2x2.8mm_Round_ROTATED
- added R1: 1K5, Resistor_SMD:R_0805_2012Metric_Pad1.20x1.40mm_HandSolder, F.Cu at (389.3, 390.2)
- added U3: TUSB4041I, Package_QFP:HTQFP-64-1EP_10x10mm_P0.5mm_EP8x8mm_Mask4.4x4.4mm_ThermalVias, F.Cu at (379.7, 389.1)
- D1, D10, D11, D12, D13, D14, D15, D16, D17, D18, D2, D3, D37, D38, D39, D4, D40, D41, D42, D43, D44, D45, D46, D47, D48, D49, D5, D50, D51, D52, D53, D54, D6, D7, D73, D74, D75, D76, D77, D78, D79, D8, D80, D81, D82, D83, D84, D85, D86, D87, D88, D89, D9, D90: value SK6812MINI-E -> D; footprint custom symbols and footprints:SK6812MINI_3535_6028_3.2x2.8mm_Round_ROTATED -> Diode_SMD:D_0805_2012Metric_Pad1.15x1.40mm_HandSolder
- D99: value D -> BAT60A; footprint Diode_SMD:D_0805_2012Metric_Pad1.15x1.40mm_HandSolder -> Diode_SMD:D_SOD-323; moved to F.Cu
- J1: moved to F.Cu
- moved D72 335.1 mm to (162.7, 328.6)
- moved D89 323.9 mm to (153.2, 347.7), turned to 270 degrees
- moved D90 319.2 mm to (177.0, 347.7), turned to 270 degrees
- moved D98 179.9 mm to (464.3, 347.4)
- moved D97 173.4 mm to (436.6, 352.4)
- moved D95 173.4 mm to (398.5, 352.4)
- moved D96 173.4 mm to (417.5, 352.4)
- moved D94 166.7 mm to (372.3, 352.4)
- moved D93 162.4 mm to (348.5, 352.7)
- moved D99 125.3 mm to (396.9, 383.4), turned to 0 degrees
- moved D92 109.0 mm to (272.3, 347.7)
- moved D91 72.9 mm to (200.8, 347.7)
- moved D85 63.8 mm to (441.3, 328.6), turned to 270 degrees
- moved D88 62.9 mm to (495.4, 350.0), turned to 90 degrees
- moved D84 61.8 mm to (417.5, 333.4), turned to 270 degrees
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Connections:
- net DN renamed DN1
- D1 pad 1: +5V -> row0
- D10 pad 1: +5V -> row0
- D11 pad 1: +5V -> row0
- D12 pad 1: +5V -> row0
- D13 pad 1: +5V -> row0
- D14 pad 1: +5V -> row0
- D15 pad 1: +5V -> row0
- D16 pad 1: +5V -> row0
- D17 pad 1: +5V -> row0
- D18 pad 1: +5V -> row0
- D19 pad 1: row0 -> row1
- D2 pad 1: +5V -> row0
- D20 pad 1: row0 -> row1
- D21 pad 1: row0 -> row1
- D22 pad 1: row0 -> row1
- D23 pad 1: row0 -> row1
- D24 pad 1: row0 -> row1
- D25 pad 1: row0 -> row1
- D26 pad 1: row0 -> row1
- D27 pad 1: row0 -> row1
- D28 pad 1: row0 -> row1
- D29 pad 1: row0 -> row1
- D3 pad 1: +5V -> row0
- D30 pad 1: row0 -> row1
- D31 pad 1: row0 -> row1
- D32 pad 1: row0 -> row1
- D33 pad 1: row0 -> row1
- D34 pad 1: row0 -> row1
- D35 pad 1: row0 -> row1
- D36 pad 1: row0 -> row1
- D37 pad 1: +5V -> row2
- D38 pad 1: +5V -> row2
- D39 pad 1: +5V -> row2
- D4 pad 1: +5V -> row0
- D40 pad 1: +5V -> row2
- D41 pad 1: +5V -> row2
- D42 pad 1: +5V -> row2
- D43 pad 1: +5V -> row2
- D44 pad 1: +5V -> row2
- D45 pad 1: +5V -> row2
- D46 pad 1: +5V -> row2
- D47 pad 1: +5V -> row2
- D48 pad 1: +5V -> row2
- D49 pad 1: +5V -> row2
- D5 pad 1: +5V -> row0
- D50 pad 1: +5V -> row2
- D51 pad 1: +5V -> row2
- D52 pad 1: +5V -> row2
- D53 pad 1: +5V -> row2
- D54 pad 1: +5V -> row2
- D54 pad 2: Net-(D1-Pad4) -> Net-(D54-Pad2)
- D55 pad 1: row1 -> row3
- D56 pad 1: row1 -> row3
- D57 pad 1: row1 -> row3
- D58 pad 1: row1 -> row3
- D59 pad 1: row1 -> row3
- D6 pad 1: +5V -> row0
- D60 pad 1: row1 -> row3
- D61 pad 1: row1 -> row3
- D62 pad 1: row1 -> row3
- D63 pad 1: row1 -> row3
- D64 pad 1: row1 -> row3
- D65 pad 1: row1 -> row3
- D66 pad 1: row1 -> row3
- D67 pad 1: row1 -> row3
- D68 pad 1: row1 -> row3
- D69 pad 1: row1 -> row3
- D7 pad 1: +5V -> row0
- D70 pad 1: row1 -> row3
- D71 pad 1: row1 -> row3
- D72 pad 1: row1 -> row4
- D73 pad 1: +5V -> row4
- D74 pad 1: +5V -> row4
- D75 pad 1: +5V -> row4
- D76 pad 1: +5V -> row4
- D77 pad 1: +5V -> row4
- D78 pad 1: +5V -> row4
- D79 pad 1: +5V -> row4
- D8 pad 1: +5V -> row0
- D80 pad 1: +5V -> row4
- D81 pad 1: +5V -> row4
- D82 pad 1: +5V -> row4
- D83 pad 1: +5V -> row4
- D84 pad 1: +5V -> row4
- D85 pad 1: +5V -> row4
- D86 pad 1: +5V -> row4
- D87 pad 1: +5V -> row4
- D88 pad 1: +5V -> row4
- D89 pad 1: +5V -> row5
- D9 pad 1: +5V -> row0
- D9 pad 2: Net-(D10-Pad4) -> Net-(D9-Pad2)
- D90 pad 1: +5V -> row5
- D90 pad 2: Net-(D37-Pad4) -> Net-(D90-Pad2)
- D91 pad 1: row2 -> row5
- D92 pad 1: row2 -> row5
- D93 pad 1: row2 -> row5
- D94 pad 1: row2 -> row5
- D95 pad 1: row2 -> row5
- D96 pad 1: row2 -> row5
- D97 pad 1: row2 -> row5
- D98 pad 1: row2 -> row5
- D99 pad 1: row2 -> +5V
- J1 pad 1: Net-(D198-Pad2) -> Net-(D99-Pad2)
- J1 pad 3: DP -> DP1
- SW1 pad 2: Net-(D19-Pad2) -> Net-(D1-Pad2)
- SW10 pad 2: Net-(D28-Pad2) -> Net-(D10-Pad2)
- SW11 pad 2: Net-(D29-Pad2) -> Net-(D11-Pad2)
- SW12 pad 2: Net-(D30-Pad2) -> Net-(D12-Pad2)
- SW13 pad 2: Net-(D31-Pad2) -> Net-(D13-Pad2)
- SW14 pad 2: Net-(D32-Pad2) -> Net-(D14-Pad2)
- SW15 pad 2: Net-(D33-Pad2) -> Net-(D15-Pad2)
- SW16 pad 2: Net-(D34-Pad2) -> Net-(D16-Pad2)
- SW17 pad 2: Net-(D35-Pad2) -> Net-(D17-Pad2)
- SW18 pad 2: Net-(D36-Pad2) -> Net-(D18-Pad2)
- SW19 pad 2: Net-(D55-Pad2) -> Net-(D19-Pad2)
- SW2 pad 2: Net-(D20-Pad2) -> Net-(D2-Pad2)
- SW20 pad 2: Net-(D56-Pad2) -> Net-(D20-Pad2)
- SW21 pad 2: Net-(D57-Pad2) -> Net-(D21-Pad2)
- SW22 pad 2: Net-(D58-Pad2) -> Net-(D22-Pad2)
- SW23 pad 2: Net-(D59-Pad2) -> Net-(D23-Pad2)
- SW24 pad 2: Net-(D60-Pad2) -> Net-(D24-Pad2)
- SW25 pad 2: Net-(D61-Pad2) -> Net-(D25-Pad2)
- SW26 pad 2: Net-(D62-Pad2) -> Net-(D26-Pad2)
- SW27 pad 2: Net-(D63-Pad2) -> Net-(D27-Pad2)
- SW28 pad 2: Net-(D64-Pad2) -> Net-(D28-Pad2)
- SW29 pad 2: Net-(D65-Pad2) -> Net-(D29-Pad2)
- SW3 pad 2: Net-(D21-Pad2) -> Net-(D3-Pad2)
- SW30 pad 2: Net-(D66-Pad2) -> Net-(D30-Pad2)
- SW31 pad 2: Net-(D67-Pad2) -> Net-(D31-Pad2)
- SW32 pad 2: Net-(D68-Pad2) -> Net-(D32-Pad2)
- SW33 pad 2: Net-(D69-Pad2) -> Net-(D33-Pad2)
- SW34 pad 2: Net-(D70-Pad2) -> Net-(D34-Pad2)
- SW35 pad 2: Net-(D71-Pad2) -> Net-(D35-Pad2)
- SW36 pad 2: Net-(D72-Pad2) -> Net-(D36-Pad2)
- SW37 pad 2: Net-(D91-Pad2) -> Net-(D37-Pad2)
- SW38 pad 2: Net-(D92-Pad2) -> Net-(D38-Pad2)
- SW39 pad 2: Net-(D93-Pad2) -> Net-(D39-Pad2)
- SW4 pad 2: Net-(D22-Pad2) -> Net-(D4-Pad2)
- SW40 pad 2: Net-(D94-Pad2) -> Net-(D40-Pad2)
- SW41 pad 2: Net-(D95-Pad2) -> Net-(D41-Pad2)
- SW42 pad 2: Net-(D96-Pad2) -> Net-(D42-Pad2)
- SW43 pad 2: Net-(D97-Pad2) -> Net-(D43-Pad2)
- SW44 pad 2: Net-(D98-Pad2) -> Net-(D44-Pad2)
- SW45 pad 2: Net-(D99-Pad2) -> Net-(D45-Pad2)
- SW46 pad 2: Net-(D100-Pad2) -> Net-(D46-Pad2)
- SW47 pad 2: Net-(D101-Pad2) -> Net-(D47-Pad2)
- SW48 pad 2: Net-(D102-Pad2) -> Net-(D48-Pad2)
- SW49 pad 2: Net-(D103-Pad2) -> Net-(D49-Pad2)
- SW5 pad 2: Net-(D23-Pad2) -> Net-(D5-Pad2)
- SW50 pad 2: Net-(D104-Pad2) -> Net-(D50-Pad2)
- SW51 pad 2: Net-(D105-Pad2) -> Net-(D51-Pad2)
- SW52 pad 2: Net-(D106-Pad2) -> Net-(D52-Pad2)
- SW53 pad 2: Net-(D107-Pad2) -> Net-(D53-Pad2)
- SW54 pad 2: Net-(D108-Pad2) -> Net-(D54-Pad2)
- SW55 pad 2: Net-(D126-Pad2) -> Net-(D55-Pad2)
- SW56 pad 2: Net-(D127-Pad2) -> Net-(D56-Pad2)
- SW57 pad 2: Net-(D128-Pad2) -> Net-(D57-Pad2)
- SW58 pad 2: Net-(D129-Pad2) -> Net-(D58-Pad2)
- SW59 pad 2: Net-(D130-Pad2) -> Net-(D59-Pad2)
- SW6 pad 2: Net-(D24-Pad2) -> Net-(D6-Pad2)
- SW60 pad 2: Net-(D131-Pad2) -> Net-(D60-Pad2)
- SW61 pad 2: Net-(D132-Pad2) -> Net-(D61-Pad2)
- SW62 pad 2: Net-(D133-Pad2) -> Net-(D62-Pad2)
- SW63 pad 2: Net-(D134-Pad2) -> Net-(D63-Pad2)
- SW64 pad 2: Net-(D135-Pad2) -> Net-(D64-Pad2)
- SW65 pad 2: Net-(D136-Pad2) -> Net-(D65-Pad2)
- SW66 pad 2: Net-(D137-Pad2) -> Net-(D66-Pad2)
- SW67 pad 2: Net-(D138-Pad2) -> Net-(D67-Pad2)
- SW68 pad 2: Net-(D139-Pad2) -> Net-(D68-Pad2)
- SW69 pad 2: Net-(D140-Pad2) -> Net-(D69-Pad2)
- SW7 pad 2: Net-(D25-Pad2) -> Net-(D7-Pad2)
- SW70 pad 2: Net-(D141-Pad2) -> Net-(D70-Pad2)
- SW71 pad 2: Net-(D142-Pad2) -> Net-(D71-Pad2)
- SW72 pad 2: Net-(D160-Pad2) -> Net-(D72-Pad2)
- SW73 pad 2: Net-(D161-Pad2) -> Net-(D73-Pad2)
- SW74 pad 2: Net-(D162-Pad2) -> Net-(D74-Pad2)
- SW75 pad 2: Net-(D163-Pad2) -> Net-(D75-Pad2)
- SW76 pad 2: Net-(D164-Pad2) -> Net-(D76-Pad2)
- SW77 pad 2: Net-(D165-Pad2) -> Net-(D77-Pad2)
- SW78 pad 2: Net-(D166-Pad2) -> Net-(D78-Pad2)
- SW79 pad 2: Net-(D167-Pad2) -> Net-(D79-Pad2)
- SW8 pad 2: Net-(D26-Pad2) -> Net-(D8-Pad2)
- SW80 pad 2: Net-(D168-Pad2) -> Net-(D80-Pad2)
- SW81 pad 2: Net-(D169-Pad2) -> Net-(D81-Pad2)
- SW82 pad 2: Net-(D170-Pad2) -> Net-(D82-Pad2)
- SW83 pad 2: Net-(D171-Pad2) -> Net-(D83-Pad2)
- SW84 pad 2: Net-(D172-Pad2) -> Net-(D84-Pad2)
- SW85 pad 2: Net-(D173-Pad2) -> Net-(D85-Pad2)
- SW86 pad 2: Net-(D174-Pad2) -> Net-(D86-Pad2)
- SW87 pad 2: Net-(D175-Pad2) -> Net-(D87-Pad2)
- SW88 pad 2: Net-(D176-Pad2) -> Net-(D88-Pad2)
- SW89 pad 2: Net-(D187-Pad2) -> Net-(D89-Pad2)
- SW9 pad 2: Net-(D27-Pad2) -> Net-(D9-Pad2)
- SW90 pad 2: Net-(D188-Pad2) -> Net-(D90-Pad2)
- SW91 pad 2: Net-(D189-Pad2) -> Net-(D91-Pad2)
- SW92 pad 2: Net-(D190-Pad2) -> Net-(D92-Pad2)
- SW93 pad 2: Net-(D191-Pad2) -> Net-(D93-Pad2)
- SW94 pad 2: Net-(D192-Pad2) -> Net-(D94-Pad2)
- SW95 pad 2: Net-(D193-Pad2) -> Net-(D95-Pad2)
- SW96 pad 2: Net-(D194-Pad2) -> Net-(D96-Pad2)
- SW97 pad 2: Net-(D195-Pad2) -> Net-(D97-Pad2)
- SW98 pad 2: Net-(D196-Pad2) -> Net-(D98-Pad2)
- U1 pad 33: DP -> DP1
Routing:
- net row0: track 347.8 -> 1948.8 mm, vias 0 -> 4
- net row1: track 346.9 -> 1536.9 mm, vias 0 -> 4
- net row2: track 337.6 -> 1132.8 mm, vias 0 -> 3
- net row3: track 339.5 -> 738.5 mm, vias 0 -> 3
- net Net-(D109-Pad4): track 378.6 -> 0.00 mm
- net Net-(D1-Pad4): track 374.6 -> 0.00 mm
- net Net-(D37-Pad4): track 370.7 -> 0.00 mm
- net Net-(D125-Pad2): track 365.4 -> 0.00 mm
- net Net-(D143-Pad4): track 335.1 -> 0.00 mm
- net row4: track 338.9 -> 599.7 mm, vias 0 -> 3
- net row5: track 318.4 -> 76.5 mm, vias 0 -> 1
- net Net-(D177-Pad4): track 88.4 -> 0.00 mm
- net Net-(D180-Pad2): track 82.4 -> 0.00 mm
- net Net-(D179-Pad2): track 66.8 -> 0.00 mm
- net Net-(D121-Pad2): track 31.1 -> 0.00 mm
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