File: GCSv1/matrix.sch (KiCad schematic (older format))
At the start: 48 parts

Commit message: Unit A and Unit B btw :)
tried to finish matrix schematic but the fucking custom symbol is dogshit
Parts:
- removed D? (x15): D, symbol Device:D
- removed LED? (x16): SK6812mini2, symbol custom:SK6812mini2
- removed SW? (x15): switch, symbol custom:switch
- added C1, C2, C3, C4, C5, C6: 100µF, symbol Device:C
- added D1, D10, D109, D11, D110, D111, D112, D113, D114, D115, D116, D117, D118, D119, D12, D120, D121, D122, D123, D124, D125, D13, D14, D143, D144, D145, D146, D147, D148, D149, D15, D150, D151, D152, D153, D154, D155, D156, D157, D158, D159, D16, D17, D177, D178, D179, D18, D180, D181, D182, D183, D184, D185, D186, D2, D3, D37, D38, D39, D4, D40, D41, D42, D43, D44, D45, D46, D47, D48, D49, D5, D50, D51, D52, D53, D54, D6, D7, D73, D74, D75, D76, D77, D78, D79, D8, D80, D81, D82, D83, D84, D85, D86, D87, D88, D89, D9, D90: SK6812MINI-E, acheron_Components:SK6812MINI_3535_6028_3.2x2.8mm_Round, symbol acheronSymbols:SK6812MINI-E
- added D100, D101, D102, D103, D104, D105, D106, D107, D108, D126, D127, D128, D129, D130, D131, D132, D133, D134, D135, D136, D137, D138, D139, D140, D141, D142, D160, D161, D162, D163, D164, D165, D166, D167, D168, D169, D170, D171, D172, D173, D174, D175, D176, D187, D188, D189, D190, D191, D192, D193, D194, D195, D196, D20, D21, D22, D23, D24, D25, D26, D27, D28, D29, D30, D31, D32, D33, D34, D35, D36, D55, D56, D57, D58, D59, D60, D61, D62, D63, D64, D65, D66, D67, D68, D69, D70, D71, D72, D91, D92, D93, D94, D95, D96, D97, D98, D99: D, symbol Device:D
- added R1: 0.5K, symbol Device:R
- added SW1, SW10, SW11, SW12, SW13, SW14, SW15, SW16, SW17, SW18, SW19, SW2, SW20, SW21, SW22, SW23, SW24, SW25, SW26, SW27, SW28, SW29, SW3, SW30, SW31, SW32, SW33, SW34, SW35, SW36, SW37, SW38, SW39, SW4, SW40, SW41, SW42, SW43, SW44, SW45, SW46, SW47, SW48, SW49, SW5, SW6, SW7, SW8, SW9: switch, symbol custom:switch
- gave numbers to parts that had none: 2
Connections:
- net labels added: LED
- wire segments 172 -> 828
- no-connect marks 0 -> 1
Other:
- moved on the sheet: D19

Commit message: fixed switches in matrix, ready for layout
Parts:
- removed SW1 (x2), SW10, SW11, SW12, SW13, SW14, SW15, SW16, SW17, SW18, SW19, SW2, SW20, SW21, SW22, SW23, SW24, SW25, SW26, SW27, SW28, SW29, SW3, SW30, SW31, SW32, SW33, SW34, SW35, SW36, SW37, SW38, SW39, SW4, SW40, SW41, SW42, SW43, SW44, SW45, SW46, SW47, SW48, SW49, SW5, SW6, SW7, SW8, SW9: switch, symbol custom:switch
- added SW1, SW10, SW11, SW12, SW13, SW15, SW16, SW17, SW18, SW19, SW2, SW20, SW21, SW22, SW23, SW24, SW25, SW26, SW27, SW28, SW29, SW3, SW30, SW31, SW33, SW34, SW35, SW36, SW38, SW39, SW4, SW40, SW41, SW42, SW43, SW44, SW45, SW46, SW47, SW48, SW49, SW5, SW51, SW52, SW53, SW54, SW56, SW57, SW58, SW59, SW6, SW60, SW61, SW62, SW63, SW64, SW65, SW66, SW68, SW69, SW7, SW70, SW71, SW73, SW74, SW75, SW76, SW77, SW78, SW79, SW8, SW80, SW81, SW82, SW84, SW85, SW86, SW87, SW9, SW95, SW96, SW97, SW98: SW_MEC_5G, MX_Alps_Hybrid:MX-1U-NoLED, symbol Switch:SW_MEC_5G
- added SW14: DEL, MX_Alps_Hybrid:MX-1.5U-NoLED, symbol Switch:SW_MEC_5G
- added SW32: BKSPC, MX_Alps_Hybrid:MX-2U-NoLED, symbol Switch:SW_MEC_5G
- added SW37: TAB, MX_Alps_Hybrid:MX-1.5U-NoLED, symbol Switch:SW_MEC_5G
- added SW50: BSLSH, MX_Alps_Hybrid:MX-1.5U-NoLED, symbol Switch:SW_MEC_5G
- added SW55: CAPS, MX_Alps_Hybrid:MX-1.75U-NoLED, symbol Switch:SW_MEC_5G
- added SW67: ENTER, MX_Alps_Hybrid:MX-2.25U-NoLED, symbol Switch:SW_MEC_5G
- added SW72: LSHFT, MX_Alps_Hybrid:MX-2.25U-NoLED, symbol Switch:SW_MEC_5G
- added SW83: RSHFT, MX_Alps_Hybrid:MX-1.5U-NoLED, symbol Switch:SW_MEC_5G
- added SW88: NUMEN, MX_Alps_Hybrid:MX-2U-NoLED, symbol Switch:SW_MEC_5G
- added SW89: CTRL, MX_Alps_Hybrid:MX-1.25U-NoLED, symbol Switch:SW_MEC_5G
- added SW90: WIN, MX_Alps_Hybrid:MX-1.25U-NoLED, symbol Switch:SW_MEC_5G
- added SW91: ALT, MX_Alps_Hybrid:MX-1.25U-NoLED, symbol Switch:SW_MEC_5G
- added SW92: SPACE, MX_Alps_Hybrid:MX-6.25U-NoLED, symbol Switch:SW_MEC_5G
- added SW93: HOME, MX_Alps_Hybrid:MX-1.25U-NoLED, symbol Switch:SW_MEC_5G
- added SW94: END, MX_Alps_Hybrid:MX-1.25U-NoLED, symbol Switch:SW_MEC_5G
- C1, C2, C3, C4, C5, C6: footprint (none) -> Capacitor_SMD:C_0805_2012Metric_Pad1.18x1.45mm_HandSolder
- D100, D101, D102, D103, D104, D105, D106, D107, D108, D126, D127, D128, D129, D130, D131, D132, D133, D134, D135, D136, D137, D138, D139, D140, D141, D142, D160, D161, D162, D163, D164, D165, D166, D167, D168, D169, D170, D171, D172, D173, D174, D175, D176, D187, D188, D189, D19, D190, D191, D192, D193, D194, D195, D196, D20, D21, D22, D23, D24, D25, D26, D27, D28, D29, D30, D31, D32, D33, D34, D35, D36, D55, D56, D57, D58, D59, D60, D61, D62, D63, D64, D65, D66, D67, D68, D69, D70, D71, D72, D91, D92, D93, D94, D95, D96, D97, D98, D99: footprint (none) -> Diode_SMD:D_0805_2012Metric_Pad1.15x1.40mm_HandSolder
- R1: footprint (none) -> Resistor_SMD:R_0805_2012Metric_Pad1.20x1.40mm_HandSolder

Commit message: pick-and-place simulator
Parts:
- SW1: value SW_MEC_5G -> ESC
- SW10: value SW_MEC_5G -> F9
- SW11: value SW_MEC_5G -> F10
- SW12: value SW_MEC_5G -> F11
- SW13: value SW_MEC_5G -> F12
- SW15: value SW_MEC_5G -> F13
- SW16: value SW_MEC_5G -> F14
- SW17: value SW_MEC_5G -> F15
- SW18: value SW_MEC_5G -> F16
- SW19: value SW_MEC_5G -> TILDE
- SW2: value SW_MEC_5G -> F1
- SW20: value SW_MEC_5G -> 1
- SW21: value SW_MEC_5G -> 2
- SW22: value SW_MEC_5G -> 3
- SW23: value SW_MEC_5G -> 4
- SW24: value SW_MEC_5G -> 5
- SW25: value SW_MEC_5G -> 6
- SW26: value SW_MEC_5G -> 7
- SW27: value SW_MEC_5G -> 8
- SW28: value SW_MEC_5G -> 9
- SW29: value SW_MEC_5G -> 0
- SW3: value SW_MEC_5G -> F2
- SW30: value SW_MEC_5G -> DASH
- SW31: value SW_MEC_5G -> EQUAL
- SW33: value SW_MEC_5G -> MOP1
- SW34: value SW_MEC_5G -> MOP2
- SW35: value SW_MEC_5G -> MOP3
- SW36: value SW_MEC_5G -> MOP4
- SW4: value SW_MEC_5G -> F3
- SW5: value SW_MEC_5G -> F4
- SW6: value SW_MEC_5G -> F5
- SW7: value SW_MEC_5G -> F6
- SW8: value SW_MEC_5G -> F7
- SW9: value SW_MEC_5G -> F8
- SW98: value SW_MEC_5G -> NUM0; footprint MX_Alps_Hybrid:MX-1U-NoLED -> MX_Alps_Hybrid:MX-2U-NoLED

Commit message: finished placing switches
Parts:
- SW38: value SW_MEC_5G -> Q
- SW39: value SW_MEC_5G -> W
- SW40: value SW_MEC_5G -> E
- SW41: value SW_MEC_5G -> R
- SW42: value SW_MEC_5G -> T
- SW43: value SW_MEC_5G -> Y
- SW44: value SW_MEC_5G -> U
- SW45: value SW_MEC_5G -> I
- SW46: value SW_MEC_5G -> O
- SW47: value SW_MEC_5G -> P
- SW48: value SW_MEC_5G -> LBRKT
- SW49: value SW_MEC_5G -> RBRKT
- SW51: value SW_MEC_5G -> NUM7
- SW52: value SW_MEC_5G -> NUM8
- SW53: value SW_MEC_5G -> NUM9
- SW54: value SW_MEC_5G -> MOP5
- SW56: value SW_MEC_5G -> A
- SW57: value SW_MEC_5G -> S
- SW58: value SW_MEC_5G -> D
- SW59: value SW_MEC_5G -> F
- SW60: value SW_MEC_5G -> G
- SW61: value SW_MEC_5G -> H
- SW62: value SW_MEC_5G -> J
- SW63: value SW_MEC_5G -> K
- SW64: value SW_MEC_5G -> L
- SW65: value SW_MEC_5G -> SMCLN
- SW66: value SW_MEC_5G -> APOST
- SW68: value SW_MEC_5G -> NUM4
- SW69: value SW_MEC_5G -> NUM5
- SW70: value SW_MEC_5G -> NUM6
- SW71: value SW_MEC_5G -> MOP6
- SW73: value SW_MEC_5G -> Z
- SW74: value SW_MEC_5G -> X
- SW75: value SW_MEC_5G -> C
- SW76: value SW_MEC_5G -> V
- SW77: value SW_MEC_5G -> B
- SW78: value SW_MEC_5G -> N
- SW79: value SW_MEC_5G -> M
- SW80: value SW_MEC_5G -> COMMA
- SW81: value SW_MEC_5G -> PRD
- SW82: value SW_MEC_5G -> SLSH
- SW84: value SW_MEC_5G -> UP
- SW85: value SW_MEC_5G -> NUM1
- SW86: value SW_MEC_5G -> NUM2
- SW87: value SW_MEC_5G -> NUM3
- SW95: value SW_MEC_5G -> LEFT
- SW96: value SW_MEC_5G -> DOWN
- SW97: value SW_MEC_5G -> RIGHT

Commit message: another backup before changing rgb symbol
Parts:
- SW1, SW10, SW11, SW12, SW13, SW14, SW15, SW16, SW17, SW18, SW19, SW2, SW20, SW21, SW22, SW23, SW24, SW25, SW26, SW27, SW28, SW29, SW3, SW30, SW31, SW32, SW33, SW34, SW35, SW36, SW37, SW38, SW39, SW4, SW40, SW41, SW42, SW43, SW44, SW45, SW46, SW47, SW48, SW49, SW5, SW50, SW51, SW52, SW53, SW54, SW55, SW56, SW57, SW58, SW59, SW6, SW60, SW61, SW62, SW63, SW64, SW65, SW66, SW67, SW68, SW69, SW7, SW70, SW71, SW72, SW73, SW74, SW75, SW76, SW77, SW78, SW79, SW8, SW80, SW81, SW82, SW83, SW84, SW85, SW86, SW87, SW88, SW89, SW9, SW90, SW91, SW92, SW93, SW94, SW95, SW96, SW97, SW98: symbol Switch:SW_MEC_5G -> custom:SW_DIP_x01_flipped
Connections:
- net col00: now also SW1.1, SW19.1, SW37.1, SW55.1, SW72.1, SW89.1; no longer SW1.3 (B), SW1.4 (B), SW19.3 (B), SW19.4 (B), SW37.3 (B), SW37.4 (B), SW55.3 (B), SW55.4 (B), SW72.3 (B), SW72.4 (B), SW89.3 (B), SW89.4 (B)
- net col01: now also SW2.1, SW20.1, SW38.1, SW56.1, SW73.1, SW90.1; no longer SW2.3 (B), SW2.4 (B), SW20.3 (B), SW20.4 (B), SW38.3 (B), SW38.4 (B), SW56.3 (B), SW56.4 (B), SW73.3 (B), SW73.4 (B), SW90.3 (B), SW90.4 (B)
- net col02: now also SW21.1, SW3.1, SW39.1, SW57.1, SW74.1, SW91.1; no longer SW21.3 (B), SW21.4 (B), SW3.3 (B), SW3.4 (B), SW39.3 (B), SW39.4 (B), SW57.3 (B), SW57.4 (B), SW74.3 (B), SW74.4 (B), SW91.3 (B), SW91.4 (B)
- net col03: now also SW22.1, SW4.1, SW40.1, SW58.1, SW75.1; no longer SW22.3 (B), SW22.4 (B), SW4.3 (B), SW4.4 (B), SW40.3 (B), SW40.4 (B), SW58.3 (B), SW58.4 (B), SW75.3 (B), SW75.4 (B)
- net col04: now also SW23.1, SW41.1, SW5.1, SW59.1, SW76.1; no longer SW23.3 (B), SW23.4 (B), SW41.3 (B), SW41.4 (B), SW5.3 (B), SW5.4 (B), SW59.3 (B), SW59.4 (B), SW76.3 (B), SW76.4 (B)
- net col05: now also SW24.1, SW42.1, SW6.1, SW60.1, SW77.1, SW92.1; no longer SW24.3 (B), SW24.4 (B), SW42.3 (B), SW42.4 (B), SW6.3 (B), SW6.4 (B), SW60.3 (B), SW60.4 (B), SW77.3 (B), SW77.4 (B), SW92.3 (B), SW92.4 (B)
- net col06: now also SW25.1, SW43.1, SW61.1, SW7.1, SW78.1; no longer SW25.3 (B), SW25.4 (B), SW43.3 (B), SW43.4 (B), SW61.3 (B), SW61.4 (B), SW7.3 (B), SW7.4 (B), SW78.3 (B), SW78.4 (B)
- net col07: now also SW26.1, SW44.1, SW62.1, SW79.1, SW8.1; no longer SW26.3 (B), SW26.4 (B), SW44.3 (B), SW44.4 (B), SW62.3 (B), SW62.4 (B), SW79.3 (B), SW79.4 (B), SW8.3 (B), SW8.4 (B)
- net col08: now also SW27.1, SW45.1, SW63.1, SW80.1, SW9.1; no longer SW27.3 (B), SW27.4 (B), SW45.3 (B), SW45.4 (B), SW63.3 (B), SW63.4 (B), SW80.3 (B), SW80.4 (B), SW9.3 (B), SW9.4 (B)
- net col09: now also SW10.1, SW28.1, SW46.1, SW64.1, SW81.1, SW93.1; no longer SW10.3 (B), SW10.4 (B), SW28.3 (B), SW28.4 (B), SW46.3 (B), SW46.4 (B), SW64.3 (B), SW64.4 (B), SW81.3 (B), SW81.4 (B), SW93.3 (B), SW93.4 (B)
- net col10: now also SW11.1, SW29.1, SW47.1, SW65.1, SW82.1, SW94.1; no longer SW11.3 (B), SW11.4 (B), SW29.3 (B), SW29.4 (B), SW47.3 (B), SW47.4 (B), SW65.3 (B), SW65.4 (B), SW82.3 (B), SW82.4 (B), SW94.3 (B), SW94.4 (B)
- net col11: now also SW12.1, SW30.1, SW48.1, SW66.1, SW83.1, SW95.1; no longer SW12.3 (B), SW12.4 (B), SW30.3 (B), SW30.4 (B), SW48.3 (B), SW48.4 (B), SW66.3 (B), SW66.4 (B), SW83.3 (B), SW83.4 (B), SW95.3 (B), SW95.4 (B)
- net col12: now also SW13.1, SW31.1, SW49.1; no longer SW13.3 (B), SW13.4 (B), SW31.3 (B), SW31.4 (B), SW49.3 (B), SW49.4 (B)
- net col13: now also SW14.1, SW32.1, SW50.1, SW67.1, SW84.1, SW96.1; no longer SW14.3 (B), SW14.4 (B), SW32.3 (B), SW32.4 (B), SW50.3 (B), SW50.4 (B), SW67.3 (B), SW67.4 (B), SW84.3 (B), SW84.4 (B), SW96.3 (B), SW96.4 (B)
- net col14: now also SW15.1, SW33.1, SW51.1, SW68.1, SW85.1, SW97.1; no longer SW15.3 (B), SW15.4 (B), SW33.3 (B), SW33.4 (B), SW51.3 (B), SW51.4 (B), SW68.3 (B), SW68.4 (B), SW85.3 (B), SW85.4 (B), SW97.3 (B), SW97.4 (B)
- net col15: now also SW16.1, SW34.1, SW52.1, SW69.1, SW86.1; no longer SW16.3 (B), SW16.4 (B), SW34.3 (B), SW34.4 (B), SW52.3 (B), SW52.4 (B), SW69.3 (B), SW69.4 (B), SW86.3 (B), SW86.4 (B)
- net col16: now also SW17.1, SW35.1, SW53.1, SW70.1, SW87.1, SW98.1; no longer SW17.3 (B), SW17.4 (B), SW35.3 (B), SW35.4 (B), SW53.3 (B), SW53.4 (B), SW70.3 (B), SW70.4 (B), SW87.3 (B), SW87.4 (B), SW98.3 (B), SW98.4 (B)
- net col17: now also SW18.1, SW36.1, SW54.1, SW71.1, SW88.1; no longer SW18.3 (B), SW18.4 (B), SW36.3 (B), SW36.4 (B), SW54.3 (B), SW54.4 (B), SW71.3 (B), SW71.4 (B), SW88.3 (B), SW88.4 (B)
- net at D19.2 (A), SW1.2: no longer SW1.1 (A)
- net at D20.2 (A), SW2.2: no longer SW2.1 (A)
- net at D35.2 (A), SW17.2: no longer SW17.1 (A)
- net at D36.2 (A), SW18.2: no longer SW18.1 (A)
- net at D21.2 (A), SW3.2: no longer SW3.1 (A)
- net at D22.2 (A), SW4.2: no longer SW4.1 (A)
- net at D23.2 (A), SW5.2: no longer SW5.1 (A)
- net at D24.2 (A), SW6.2: no longer SW6.1 (A)
- net at D25.2 (A), SW7.2: no longer SW7.1 (A)
- net at D26.2 (A), SW8.2: no longer SW8.1 (A)
- net at D27.2 (A), SW9.2: no longer SW9.1 (A)
- net at D28.2 (A), SW10.2: no longer SW10.1 (A)
- net at D29.2 (A), SW11.2: no longer SW11.1 (A)
- net at D30.2 (A), SW12.2: no longer SW12.1 (A)
- net at D31.2 (A), SW13.2: no longer SW13.1 (A)
- net at D32.2 (A), SW14.2: no longer SW14.1 (A)
- net at D33.2 (A), SW15.2: no longer SW15.1 (A)
- net at D34.2 (A), SW16.2: no longer SW16.1 (A)
- net at D55.2 (A), SW19.2: no longer SW19.1 (A)
- net at D56.2 (A), SW20.2: no longer SW20.1 (A)
- net at D71.2 (A), SW35.2: no longer SW35.1 (A)
- net at D72.2 (A), SW36.2: no longer SW36.1 (A)
- net at D57.2 (A), SW21.2: no longer SW21.1 (A)
- net at D58.2 (A), SW22.2: no longer SW22.1 (A)
- net at D59.2 (A), SW23.2: no longer SW23.1 (A)
- net at D60.2 (A), SW24.2: no longer SW24.1 (A)
- net at D61.2 (A), SW25.2: no longer SW25.1 (A)
- net at D62.2 (A), SW26.2: no longer SW26.1 (A)
- net at D63.2 (A), SW27.2: no longer SW27.1 (A)
- net at D64.2 (A), SW28.2: no longer SW28.1 (A)
- net at D65.2 (A), SW29.2: no longer SW29.1 (A)
- net at D66.2 (A), SW30.2: no longer SW30.1 (A)
- net at D67.2 (A), SW31.2: no longer SW31.1 (A)
- net at D68.2 (A), SW32.2: no longer SW32.1 (A)
- net at D69.2 (A), SW33.2: no longer SW33.1 (A)
- net at D70.2 (A), SW34.2: no longer SW34.1 (A)
- net at D91.2 (A), SW37.2: no longer SW37.1 (A)
- net at D92.2 (A), SW38.2: no longer SW38.1 (A)
- net at D107.2 (A), SW53.2: no longer SW53.1 (A)
- net at D108.2 (A), SW54.2: no longer SW54.1 (A)
- net at D93.2 (A), SW39.2: no longer SW39.1 (A)
- net at D94.2 (A), SW40.2: no longer SW40.1 (A)
- net at D95.2 (A), SW41.2: no longer SW41.1 (A)
- net at D96.2 (A), SW42.2: no longer SW42.1 (A)
- net at D97.2 (A), SW43.2: no longer SW43.1 (A)
- net at D98.2 (A), SW44.2: no longer SW44.1 (A)
- net at D99.2 (A), SW45.2: no longer SW45.1 (A)
- net at D100.2 (A), SW46.2: no longer SW46.1 (A)
- net at D101.2 (A), SW47.2: no longer SW47.1 (A)
- net at D102.2 (A), SW48.2: no longer SW48.1 (A)
- net at D103.2 (A), SW49.2: no longer SW49.1 (A)
- net at D104.2 (A), SW50.2: no longer SW50.1 (A)
- net at D105.2 (A), SW51.2: no longer SW51.1 (A)
- net at D106.2 (A), SW52.2: no longer SW52.1 (A)
- net at D126.2 (A), SW55.2: no longer SW55.1 (A)
- net at D127.2 (A), SW56.2: no longer SW56.1 (A)
- net at D141.2 (A), SW70.2: no longer SW70.1 (A)
- net at D142.2 (A), SW71.2: no longer SW71.1 (A)
- net at D128.2 (A), SW57.2: no longer SW57.1 (A)
- net at D129.2 (A), SW58.2: no longer SW58.1 (A)
- net at D130.2 (A), SW59.2: no longer SW59.1 (A)
- net at D131.2 (A), SW60.2: no longer SW60.1 (A)
- net at D132.2 (A), SW61.2: no longer SW61.1 (A)
- net at D133.2 (A), SW62.2: no longer SW62.1 (A)
- net at D134.2 (A), SW63.2: no longer SW63.1 (A)
- net at D135.2 (A), SW64.2: no longer SW64.1 (A)
- net at D136.2 (A), SW65.2: no longer SW65.1 (A)
- net at D137.2 (A), SW66.2: no longer SW66.1 (A)
- net at D138.2 (A), SW67.2: no longer SW67.1 (A)
- net at D139.2 (A), SW68.2: no longer SW68.1 (A)
- net at D140.2 (A), SW69.2: no longer SW69.1 (A)
- net at D160.2 (A), SW72.2: no longer SW72.1 (A)
- net at D161.2 (A), SW73.2: no longer SW73.1 (A)
- net at D175.2 (A), SW87.2: no longer SW87.1 (A)
- net at D176.2 (A), SW88.2: no longer SW88.1 (A)
- net at D162.2 (A), SW74.2: no longer SW74.1 (A)
- net at D163.2 (A), SW75.2: no longer SW75.1 (A)
- net at D164.2 (A), SW76.2: no longer SW76.1 (A)
- net at D165.2 (A), SW77.2: no longer SW77.1 (A)
- net at D166.2 (A), SW78.2: no longer SW78.1 (A)
- net at D167.2 (A), SW79.2: no longer SW79.1 (A)
- net at D168.2 (A), SW80.2: no longer SW80.1 (A)
- net at D169.2 (A), SW81.2: no longer SW81.1 (A)
- net at D170.2 (A), SW82.2: no longer SW82.1 (A)
- net at D171.2 (A), SW83.2: no longer SW83.1 (A)
- net at D172.2 (A), SW84.2: no longer SW84.1 (A)
- net at D173.2 (A), SW85.2: no longer SW85.1 (A)
- net at D174.2 (A), SW86.2: no longer SW86.1 (A)
- net at D187.2 (A), SW89.2: no longer SW89.1 (A)
- net at D188.2 (A), SW90.2: no longer SW90.1 (A)
- net at D196.2 (A), SW98.2: no longer SW98.1 (A)
- net at D189.2 (A), SW91.2: no longer SW91.1 (A)
- net at D190.2 (A), SW92.2: no longer SW92.1 (A)
- net at D191.2 (A), SW93.2: no longer SW93.1 (A)
- net at D192.2 (A), SW94.2: no longer SW94.1 (A)
- net at D193.2 (A), SW95.2: no longer SW95.1 (A)
- net at D194.2 (A), SW96.2: no longer SW96.1 (A)
- net at D195.2 (A), SW97.2: no longer SW97.1 (A)
- net LED renamed LED_IN

Commit message: matrix wiring 90% done
still need to figure out how to get power to LEDs (probably route 5V through top plane, then fill in the rest of the top with ground; not much point to filling bottom plane with ground considering all the routing for rows, LED's, and other circuitry under the spacebar)

also need to get rows and columns into buses in the spacebar area, otherwise all that's left is min-maxing the positions of connector, MCU, VRM, resonator, and capacitors/resistors/diodes
Parts:
- D1, D10, D109, D11, D110, D111, D112, D113, D114, D115, D116, D117, D118, D119, D12, D120, D121, D122, D123, D124, D125, D13, D14, D143, D144, D145, D146, D147, D148, D149, D15, D150, D151, D152, D153, D154, D155, D156, D157, D158, D159, D16, D17, D177, D178, D179, D18, D180, D181, D182, D183, D184, D185, D186, D2, D3, D37, D38, D39, D4, D40, D41, D42, D43, D44, D45, D46, D47, D48, D49, D5, D50, D51, D52, D53, D54, D6, D7, D73, D74, D75, D76, D77, D78, D79, D8, D80, D81, D82, D83, D84, D85, D86, D87, D88, D89, D9, D90: footprint acheron_Components:SK6812MINI_3535_6028_3.2x2.8mm_Round -> custom symbols and footprints:SK6812MINI_3535_6028_3.2x2.8mm_Round_ROTATED

Commit message: redid matrix routing, not doing USB daughter board because of parts availability
Parts:
- removed C1, C2, C3, C4, C5, C6: 100µF, Capacitor_SMD:C_0805_2012Metric_Pad1.18x1.45mm_HandSolder, symbol Device:C
- removed D1, D10, D109, D11, D110, D111, D112, D113, D114, D115, D116, D117, D118, D119, D12, D120, D121, D122, D123, D124, D125, D13, D14, D143, D144, D145, D146, D147, D148, D149, D15, D150, D151, D152, D153, D154, D155, D156, D157, D158, D159, D16, D17, D177, D178, D179, D18, D180, D181, D182, D183, D184, D185, D186, D2, D3, D37, D38, D39, D4, D40, D41, D42, D43, D44, D45, D46, D47, D48, D49, D5, D50, D51, D52, D53, D54, D6, D7, D73, D74, D75, D76, D77, D78, D79, D8, D80, D81, D82, D83, D84, D85, D86, D87, D88, D89, D9, D90: SK6812MINI-E, custom symbols and footprints:SK6812MINI_3535_6028_3.2x2.8mm_Round_ROTATED, symbol acheronSymbols:SK6812MINI-E
- removed R1: 0.5K, Resistor_SMD:R_0805_2012Metric_Pad1.20x1.40mm_HandSolder, symbol Device:R
- renumbered D19 to D1, D28 to D10, D29 to D11, D30 to D12, D31 to D13, D32 to D14, D33 to D15, D34 to D16, D35 to D17, D36 to D18, D55 to D19, D20 to D2, D56 to D20, D57 to D21, D58 to D22, D59 to D23, D60 to D24, D61 to D25, D62 to D26, D63 to D27, D64 to D28, D65 to D29, D21 to D3, D66 to D30, D67 to D31, D68 to D32, D69 to D33, D70 to D34, D71 to D35, D72 to D36, D91 to D37, D92 to D38, D93 to D39, D22 to D4, D94 to D40, D95 to D41, D96 to D42, D97 to D43, D98 to D44, D99 to D45, D100 to D46, D101 to D47, D102 to D48, D103 to D49, D23 to D5, D104 to D50, D105 to D51, D106 to D52, D107 to D53, D108 to D54, D126 to D55, D127 to D56, D128 to D57, D129 to D58, D130 to D59, D24 to D6, D131 to D60, D132 to D61, D133 to D62, D134 to D63, D135 to D64, D136 to D65, D137 to D66, D138 to D67, D139 to D68, D140 to D69, D25 to D7, D141 to D70, D142 to D71, D160 to D72, D161 to D73, D162 to D74, D163 to D75, D164 to D76, D165 to D77, D166 to D78, D167 to D79, D26 to D8, D168 to D80, D169 to D81, D170 to D82, D171 to D83, D172 to D84, D173 to D85, D174 to D86, D175 to D87, D176 to D88, D187 to D89, D27 to D9, D188 to D90, D189 to D91, D190 to D92, D191 to D93, D192 to D94, D193 to D95, D194 to D96, D195 to D97, D196 to D98
Connections:
- no-connect marks 1 -> 0
Other:
- moved on the sheet: D1, D10, D11, D12, D13, D14, D15, D16, D17, D18, D19, D2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
